File: MicroScope/hardware/MicroScope III.kicad_pcb (KiCad board)
At the start: 2 copper layers, 38.2 x 128.3 mm, 48 parts, among them J1 Power, J2 OLED, SW1 SW_Push, SW2 SW_Push, SW3 SW_Push, SW4 SW_Push, SW5 SW_Push, U1 TL431DBZ, U2 MCP6004, U3 YAAJ_BluePill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

Commit message: Add files via upload
Parts:
- removed R2: 3k6, Resistor_SMD:R_0805_2012MetricValue
- removed U1: TL431DBZ, Package_TO_SOT_SMD:SOT-23
- R1: value 5k1 -> 6k8
- R3: value 3k -> 10k
Connections:
- R3 pad 1: Net-(R2-Pad2) -> GND
Routing:
- net Net-(R2-Pad2): track 10.5 -> 0.00 mm
- net Vref: track 50.6 -> 48.0 mm
