File: MicroScope/hardware/MicroScope III.kicad_sch (KiCad schematic)
At the start: 37 parts, among them J1 Power, J2 OLED, SW1 SW_Push, SW2 SW_Push, SW3 SW_Push, SW4 SW_Push, SW5 SW_Push, U1 TL431DBZ, U2 MCP6004, U3 YAAJ_BluePill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

Commit message: Add files via upload
Parts:
- removed R2: 3k6, Resistor_SMD:R_0805_2012MetricValue, symbol Device:R
- removed U1: TL431DBZ, Package_TO_SOT_SMD:SOT-23, symbol Reference_Voltage:TL431DBZ
- R1: value 5k1 -> 6k8
- R3: value 3k -> 10k
Connections:
- net GND: now also R3.1
Other:
- moved on the sheet: R3
Changed lines of the file:
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@@
   (junction (at 120.65 95.25) (diameter 1.016) (color 0 0 0 0))
   (junction (at 120.65 128.27) (diameter 1.016) (color 0 0 0 0))
-  (junction (at 133.35 175.26) (diameter 1.016) (color 0 0 0 0))
   (junction (at 148.59 177.8) (diameter 1.016) (color 0 0 0 0))
   (junction (at 166.37 96.52) (diameter 1.016) (color 0 0 0 0))
@@
     (stroke (width 0) (type solid) (color 0 0 0 0))
   )
-  (wire (pts (xy 133.35 175.26) (xy 146.05 175.26))
-    (stroke (width 0) (type solid) (color 0 0 0 0))
-  )
-  (wire (pts (xy 133.35 182.88) (xy 144.78 182.88))
-    (stroke (width 0) (type solid) (color 0 0 0 0))
-  )
-  (wire (pts (xy 144.78 177.8) (xy 148.59 177.8))
-    (stroke (width 0) (type solid) (color 0 0 0 0))
-  )
-  (wire (pts (xy 144.78 182.88) (xy 144.78 177.8))
-    (stroke (width 0) (type solid) (color 0 0 0 0))
-  )
   (wire (pts (xy 148.59 177.8) (xy 163.83 177.8))
     (stroke (width 0) (type solid) (color 0 0 0 0))
@@
     (pin "1")
   )
-  (symbol (lib_id "power:GND") (at 133.35 167.64 180) (unit 1)
-    (in_bom yes) (on_board yes) (fields_autoplaced)
-    (property "Reference" "#PWR0104" (id 0) (at 133.35 161.29 0)
-      (effects (font (size 1.27 1.27)) hide)
-    )
-    (property "Value" "GND" (id 1) (at 133.35 164.0926 0))
-    (property "Footprint" "" (id 2) (at 133.35 167.64 0)
-      (effects (font (size 1.27 1.27)) hide)
-    )
-    (property "Datasheet" "" (id 3) (at 133.35 167.64 0)
-      (effects (font (size 1.27 1.27)) hide)
-    )
-    (pin "1")
-  )
-  (symbol (lib_id "power:GND") (at 148.59 172.72 180) (unit 1)
-    (in_bom yes) (on_board yes) (fields_autoplaced)
-    (property "Reference" "#PWR0101" (id 0) (at 148.59 166.37 0)
-      (effects (font (size 1.27 1.27)) hide)
-    )
-    (property "Value" "GND" (id 1) (at 148.59 169.1726 0))
-    (property "Footprint" "" (id 2) (at 148.59 172.72 0)
-      (effects (font (size 1.27 1.27)) hide)
-    )
-    (property "Datasheet" "" (id 3) (at 148.59 172.72 0)
+  (symbol (lib_id "power:GND") (at 148.59 170.18 180) (unit 1)
+    (in_bom yes) (on_board yes) (fields_autoplaced)
+    (property "Reference" "#PWR0104" (id 0) (at 148.59 163.83 0)
+      (effects (font (size 1.27 1.27)) hide)
+    )
+    (property "Value" "GND" (id 1) (at 148.59 166.6326 0))
+    (property "Footprint" "" (id 2) (at 148.59 170.18 0)
+      (effects (font (size 1.27 1.27)) hide)
+    )
+    (property "Datasheet" "" (id 3) (at 148.59 170.18 0)
       (effects (font (size 1.27 1.27)) hide)
     )
@@
     (pin "2")
   )
-  (symbol (lib_id "Device:R") (at 133.35 171.45 0) (unit 1)
-    (in_bom yes) (on_board yes) (fields_autoplaced)
-    (property "Reference" "R2" (id 0) (at 135.1281 170.6891 0)
+  (symbol (lib_id "Device:R") (at 148.59 173.99 0) (unit 1)
+    (in_bom yes) (on_board yes)
+    (property "Reference" "R3" (id 0) (at 150.3681 173.2291 0)
       (effects (font (size 1.27 1.27)) (justify left))
     )
-    (property "Value" "3k6" (id 1) (at 135.1281 172.9878 0)
+    (property "Value" "10k" (id 1) (at 150.3681 175.5278 0)
       (effects (font (size 1.27 1.27)) (justify left))
     )
-    (property "Footprint" "Resistor_SMD:R_0805_2012MetricValue" (id 2) (at 131.572 171.45 90)
-      (effects (font (size 1.27 1.27)) hide)
-    )
-    (property "Datasheet" "~" (id 3) (at 133.35 171.45 0)
-      (effects (font (size 1.27 1.27)) hide)
-    )
-    (property "LCSC" "C18359" (id 4) (at 133.35 171.45 0)
-      (effects (font (size 1.27 1.27)) hide)
-    )
-    (pin "1")
-    (pin "2")
-  )
-  (symbol (lib_id "Device:R") (at 133.35 179.07 0) (unit 1)
-    (in_bom yes) (on_board yes) (fields_autoplaced)
-    (property "Reference" "R3" (id 0) (at 135.1281 178.3091 0)
-      (effects (font (size 1.27 1.27)) (justify left))
-    )
-    (property "Value" "3k" (id 1) (at 135.1281 180.6078 0)
-      (effects (font (size 1.27 1.27)) (justify left))
-    )
-    (property "Footprint" "Resistor_SMD:R_0805_2012MetricValue" (id 2) (at 131.572 179.07 90)
-      (effects (font (size 1.27 1.27)) hide)
-    )
-    (property "Datasheet" "~" (id 3) (at 133.35 179.07 0)
-      (effects (font (size 1.27 1.27)) hide)
-    )
-    (property "LCSC" "C17661" (id 4) (at 133.35 179.07 0)
+    (property "Footprint" "Resistor_SMD:R_0805_2012MetricValue" (id 2) (at 146.812 173.99 90)
+      (effects (font (size 1.27 1.27)) hide)
+    )
+    (property "Datasheet" "~" (id 3) (at 148.59 173.99 0)
+      (effects (font (size 1.27 1.27)) hide)
+    )
+    (property "LCSC" "C17661" (id 4) (at 148.59 173.99 0)
       (effects (font (size 1.27 1.27)) hide)
     )
@@
       (effects (font (size 1.27 1.27)) (justify left))
     )
-    (property "Value" "5k1" (id 1) (at 150.3681 183.1478 0)
+    (property "Value" "6k8" (id 1) (at 150.3681 183.1478 0)
       (effects (font (size 1.27 1.27)) (justify left))
     )
@@
     (pin "1")
     (pin "2")
-  )
-  (symbol (lib_id "Reference_Voltage:TL431DBZ") (at 148.59 175.26 90) (unit 1)
-    (in_bom yes) (on_board yes) (fields_autoplaced)
-    (property "Reference" "U1" (id 0) (at 150.3681 174.4991 90)
-      (effects (font (size 1.27 1.27)) (justify right))
-    )
-    (property "Value" "TL431DBZ" (id 1) (at 150.3681 176.7978 90)
-      (effects (font (size 1.27 1.27)) (justify right))
-    )
-    (property "Footprint" "Package_TO_SOT_SMD:SOT-23" (id 2) (at 152.4 175.26 0)
-      (effects (font (size 1.27 1.27) italic) hide)
-    )
-    (property "Datasheet" "http://www.ti.com/lit/ds/symlink/tl431.pdf" (id 3) (at 148.59 175.26 0)
-      (effects (font (size 1.27 1.27) italic) hide)
-    )
-    (property "LCSC" "C23892" (id 4) (at 148.59 175.26 90)
-      (effects (font (size 1.27 1.27)) hide)
-    )
-    (pin "1")
-    (pin "2")
-    (pin "3")
   )
   (symbol (lib_id "Device:C_Polarized") (at 45.72 168.91 0) (unit 1)
@@
       (reference "#PWR05") (unit 1) (value "GND") (footprint "")
     )
-    (path "/c615f9a0-481f-4b86-b111-be8e32ae3437"
-      (reference "#PWR0101") (unit 1) (value "GND") (footprint "")
-    )
     (path "/aaf183c4-9dbf-4daf-986c-d0fa5f967ad8"
       (reference "#PWR0102") (unit 1) (value "-12V") (footprint "")
@@
     )
     (path "/b52d1f18-35bd-42e2-be67-1f714ed23022"
-      (reference "R1") (unit 1) (value "5k1") (footprint "Resistor_SMD:R_0805_2012MetricValue")
-    )
-    (path "/e6698276-6802-43ea-8755-134f3bbbb437"
-      (reference "R2") (unit 1) (value "3k6") (footprint "Resistor_SMD:R_0805_2012MetricValue")
+      (reference "R1") (unit 1) (value "6k8") (footprint "Resistor_SMD:R_0805_2012MetricValue")
     )
     (path "/e6417e84-c1dc-4ce3-8277-62ee527ace81"
-      (reference "R3") (unit 1) (value "3k") (footprint "Resistor_SMD:R_0805_2012MetricValue")
+      (reference "R3") (unit 1) (value "10k") (footprint "Resistor_SMD:R_0805_2012MetricValue")
     )
     (path "/c2c6b49b-29ac-4cd4-867d-5acd7b51cdcf"
@@
       (reference "SW5") (unit 1) (value "SW_Push") (footprint "Button_Switch_THT:SW_PUSH_6mm")
     )
-    (path "/876643ab-018e-4e9e-8702-9ef52e9c2541"
-      (reference "U1") (unit 1) (value "TL431DBZ") (footprint "Package_TO_SOT_SMD:SOT-23")
-    )
     (path "/673d26e8-9283-4009-95ff-7fb26662be6d"
